Commit message: experimenting with using nav2 on custom robot. still need correct frames to be published to allow transforms.

File: resource/robot1.urdf (robot description, URDF)
Before this commit: robot robot1, 2 links, 1 joints
Links:
- link base_link: geometry collision cylinder length=0.06 radius=0.075; visual cylinder length=0.06 radius=0.075
Joints:
- joint lidar_joint: origin xyz=0 0 0.1 rpy=0 0 0 -> xyz=0 0 0.05 rpy=0 0 0

File: resource/robot2.urdf (robot description, URDF)
Before this commit: robot robot2, 2 links, 1 joints
Links:
- link base_link: geometry collision cylinder length=0.06 radius=0.075; visual cylinder length=0.06 radius=0.075
Joints:
- joint lidar_joint: origin xyz=0 0 0.1 rpy=0 0 0 -> xyz=0 0 0.05 rpy=0 0 0
